Commit message: feat: add new reward function and update URDF for robot links and meshes

File: resources/robots/pointfoot/PF_TRON1A/urdf/robot.urdf (robot description, URDF)
Before this commit: robot point_foot, 12 links, 11 joints
Links:
- link abad_L_Link: mass 1.614 -> 1.469; geometry collision cylinder length=0.05 radius=0.05; visual mesh filename=../meshes/abad_L_Link.STL
- link abad_R_Link: mass 1.614 -> 1.469; geometry collision cylinder length=0.05 radius=0.05; visual mesh filename=../meshes/abad_R_Link.STL
- link base_Link: mass 8.557 -> 9.585; geometry collision box size=0.265 0.26 0.18; visual mesh filename=../meshes/base_Link.STL
- link foot_L_Link: mass 0.157 -> 0.18; geometry collision sphere radius=0.032; visual mesh filename=../meshes/foot_L_Link.STL
- link foot_R_Link: mass 0.157 -> 0.18; geometry collision sphere radius=0.032; visual mesh filename=../meshes/foot_R_Link.STL
- link hip_L_Link: mass 2.435 -> 2.3; geometry collision cylinder length=0.18 radius=0.035; visual mesh filename=../meshes/hip_L_Link.STL
- link hip_R_Link: mass 2.435 -> 2.3; geometry collision cylinder length=0.18 radius=0.035; visual mesh filename=../meshes/hip_R_Link.STL
- link knee_L_Link: mass 0.573 -> 0.55; geometry collision cylinder length=0.26 radius=0.015; visual mesh filename=../meshes/knee_L_Link.STL
- link knee_R_Link: mass 0.573 -> 0.55; geometry collision cylinder length=0.26 radius=0.015; visual mesh filename=../meshes/knee_R_Link.STL
Joints:
- joint abad_L_Joint: limit lower=-0.38397 upper=1.39626 effort=80.0 velocity=20.0 -> lower=-0.38397 upper=1.39626 effort=80.0 velocity=15.0; origin xyz=0.01241 0.10494 -0.09876 rpy=0 0 0 -> xyz=55.56E-03 105E-03 -260.2E-03 rpy=0 0 0
- joint abad_R_Joint: limit lower=-1.39626 upper=0.38397 effort=80.0 velocity=20.0 -> lower=-1.39626 upper=0.38397 effort=80.0 velocity=15.0; origin xyz=0.01241 -0.10494 -0.09876 rpy=0 0 0 -> xyz=55.56E-03 -105E-03 -260.2E-03 rpy=0 0 0
- joint contact_L_Joint: origin xyz=0 0 -0.03 rpy=0 0 0 -> xyz=0 0 -0.032 rpy=0 0 0
- joint contact_R_Joint: origin xyz=0 0 -0.03 rpy=0 0 0 -> xyz=0 0 -0.032 rpy=0 0 0
- joint foot_L_Joint: origin xyz=0.15 0 -0.25981 rpy=0 0 0 -> xyz=0.150 0 -0.25981 rpy=0 0 0
- joint foot_R_Joint: origin xyz=0.15 0 -0.25981 rpy=0 0 0 -> xyz=0.150 0 -0.25981 rpy=0 0 0
- joint hip_L_Joint: limit lower=-1.012291 upper=1.518436 effort=80.0 velocity=20.0 -> lower=-1.012291 upper=1.396263 effort=80.0 velocity=15.0; origin xyz=-0.07696 0.02066 0 rpy=0 0 0 -> xyz=-0.077 0.02050 0 rpy=0 0 0
- joint hip_R_Joint: limit lower=-1.518436 upper=1.012291 effort=80.0 velocity=20.0 -> lower=-1.396263 upper=1.012291 effort=80.0 velocity=15.0; origin xyz=-0.07696 -0.02066 0 rpy=0 0 0 -> xyz=-0.077 -0.02050 0 rpy=0 0 0
- joint knee_L_Joint: limit lower=-0.872665 upper=1.396263 effort=80 velocity=20 -> lower=-0.872665 upper=1.361357 effort=80 velocity=15; origin xyz=-0.15004 -0.02018 -0.25981 rpy=0 0 0 -> xyz=-0.1500 -0.02050 -0.25981 rpy=0 0 0
- joint knee_R_Joint: limit lower=-1.396263 upper=0.872665 effort=80 velocity=50 -> lower=-1.361357 upper=0.872665 effort=80 velocity=15; origin xyz=-0.15004 0.02018 -0.25981 rpy=0 0 0 -> xyz=-0.1500 0.02050 -0.25981 rpy=0 0 0
